File: BPSDisplay.sch (KiCad schematic (older format))
At the start: 22 parts, among them J1 SWD, J2 Conn_02x06_Counter_Clockwise, P1 Conn_02x20_Odd_Even, SW1 Reset, U1 STM32F413RHTx, Y1 8M

Commit message: Confimred Schematic and generated Netlist
Connections:
- net DISPCS: no longer names the net of U1.50 (PA15)
- net GPIO12(PWM0): no longer names the net of P1.32 (Pin_32)
- net GPIO14(TXD0): no longer names the net of P1.8 (Pin_8)
- net GPIO15(RXD0): no longer names the net of P1.10 (Pin_10)
- net GPIO16: no longer names the net of P1.36 (Pin_36)
- net GPIO18(GEN1)(PWM0): no longer names the net of P1.12 (Pin_12)
- net GPIO2(SDA1): no longer names the net of P1.3 (Pin_3)
- net GPIO20(SPI1_MOSI): no longer names the net of P1.38 (Pin_38)
- net GPIO21(SPI1_SCK): no longer names the net of P1.40 (Pin_40)
- net GPIO22(GEN3): no longer names the net of P1.15 (Pin_15)
- net GPIO23(GEN4): no longer names the net of P1.16 (Pin_16)
- net GPIO26: no longer names the net of P1.37 (Pin_37)
- net GPIO27(GEN2): no longer names the net of P1.13 (Pin_13)
- net GPIO3(SCL1): no longer names the net of P1.5 (Pin_5)
- net GPIO4(GCLK): no longer names the net of P1.7 (Pin_7)
- net GPIO7(SPI1_CE_N): no longer names the net of P1.26 (Pin_26)
- net ID_SC: no longer names the net of P1.28 (Pin_28)
- net ID_SD: no longer names the net of P1.27 (Pin_27)
- no-connect marks 30 -> 48
Changed lines of the file:
@@
 Wire Wire Line
 	2650 2700 2650 3150
-Wire Wire Line
-	2750 1100 2750 1200
-Text Label 3600 3000 2    50   ~ 0
-GPIO21(SPI1_SCK)
-Wire Wire Line
-	2550 3000 3600 3000
 $Comp
 L Connector_Generic:Conn_02x20_Odd_Even P1
@@
 Wire Wire Line
 	2650 1300 2550 1300
-Text Label 3600 1800 2    50   ~ 0
-GPIO23(GEN4)
 Text Label 3600 1900 2    50   ~ 0
 GPIO24(GEN5)
@@
 Text Label 3600 2200 2    50   ~ 0
 GPIO8(SPI0_CE_N)
-Text Label 3600 2300 2    50   ~ 0
-GPIO7(SPI1_CE_N)
-Text Label 3600 2400 2    50   ~ 0
-ID_SC
-Text Label 3600 2600 2    50   ~ 0
-GPIO12(PWM0)
-Text Label 3600 2800 2    50   ~ 0
-GPIO16
-Text Label 3600 2900 2    50   ~ 0
-GPIO20(SPI1_MOSI)
-Text Label 900  2900 0    50   ~ 0
-GPIO26
 Text Label 900  2800 0    50   ~ 0
 GPIO19
@@
 Text Label 900  2500 0    50   ~ 0
 GPIO5
-Text Label 900  2400 0    50   ~ 0
-ID_SD
 Text Label 900  2200 0    50   ~ 0
 GPIO11(SPI0_SCK)
@@
 Text Label 900  2000 0    50   ~ 0
 GPIO10(SPI0_MOSI)
-Text Label 900  1800 0    50   ~ 0
-GPIO22(GEN3)
-Text Label 900  1700 0    50   ~ 0
-GPIO27(GEN2)
 Text Label 900  1600 0    50   ~ 0
 GPIO17(GEN0)
-Text Label 900  1400 0    50   ~ 0
-GPIO4(GCLK)
-Text Label 900  1300 0    50   ~ 0
-GPIO3(SCL1)
-Text Label 900  1200 0    50   ~ 0
-GPIO2(SDA1)
-Wire Wire Line
-	2550 2600 3600 2600
 Wire Wire Line
 	2550 1900 3600 1900
 Wire Wire Line
-	2550 1800 3600 1800
-Wire Wire Line
 	2550 2200 3600 2200
 Wire Wire Line
 	2550 2100 3600 2100
 Wire Wire Line
-	2550 2400 3600 2400
-Wire Wire Line
-	2550 2300 3600 2300
-Wire Wire Line
-	2550 2900 3600 2900
-Wire Wire Line
-	2550 2800 3600 2800
-Wire Wire Line
-	900  2900 2050 2900
-Wire Wire Line
 	900  2800 2050 2800
 Wire Wire Line
@@
 	900  2500 2050 2500
 Wire Wire Line
-	2050 2400 900  2400
-Wire Wire Line
 	900  2200 2050 2200
 Wire Wire Line
@@
 	2050 2000 900  2000
 Wire Wire Line
-	900  1800 2050 1800
-Wire Wire Line
-	900  1700 2050 1700
-Wire Wire Line
 	2050 1600 900  1600
-Wire Wire Line
-	900  1400 2050 1400
-Wire Wire Line
-	900  1300 2050 1300
-Wire Wire Line
-	2050 1200 900  1200
 Connection ~ 1950 2300
 Wire Wire Line
@@
 	1    0    0    -1
 $EndComp
-Connection ~ 2750 1100
-Wire Wire Line
-	2750 1200 2550 1200
 Wire Wire Line
 	2750 1100 2550 1100
@@
 Wire Wire Line
 	2250 3850 1900 3850
-Wire Wire Line
-	6750 3200 7250 3200
-Text Label 7250 3200 2    50   ~ 0
-DISPCS
 $Comp
 L Connector_Generic:Conn_02x06_Counter_Clockwise J2
@@
 NoConn ~ 5350 3400
 NoConn ~ 5350 3500
-Wire Wire Line
-	2550 1500 3600 1500
-Wire Wire Line
-	2550 1600 3600 1600
-Wire Wire Line
-	2550 1400 3600 1400
-Text Label 3600 1600 2    50   ~ 0
-GPIO18(GEN1)(PWM0)
-Text Label 3600 1500 2    50   ~ 0
-GPIO15(RXD0)
-Text Label 3600 1400 2    50   ~ 0
-GPIO14(TXD0)
 $Comp
 L BPSDisplay-rescue:Mounting_Hole-Mechanical MK3
@@
 	0    1    1    0
 $EndComp
+NoConn ~ 6750 3200
+NoConn ~ 2050 1200
+NoConn ~ 2050 1300
+NoConn ~ 2050 1400
+NoConn ~ 2050 1700
+NoConn ~ 2050 1800
+NoConn ~ 2050 2400
+NoConn ~ 2050 2900
+NoConn ~ 2550 3000
+NoConn ~ 2550 2900
+NoConn ~ 2550 2800
+NoConn ~ 2550 2600
+NoConn ~ 2550 2400
+NoConn ~ 2550 2300
+NoConn ~ 2550 1800
+NoConn ~ 2550 1600
+NoConn ~ 2550 1500
+NoConn ~ 2550 1400
+Wire Wire Line
+	2750 1200 2550 1200
+Connection ~ 2750 1100
+Wire Wire Line
+	2750 1100 2750 1200
 $EndSCHEMATC

Commit message: Split Logic Analyzer
& added second CAN connector
Parts:
- removed J2: Conn_02x06_Counter_Clockwise, Connector_PinHeader_2.54mm:PinHeader_2x06_P2.54mm_Vertical, symbol Connector_Generic:Conn_02x06_Counter_Clockwise
- added J6: CAN_LogicAnalyzer, symbol Connector_Generic:Conn_01x03
- added J7: SPI0_LogicAnalyzer, symbol Connector_Generic:Conn_01x05
- added J8: GEN_LogicAnalyzer, symbol Connector_Generic:Conn_01x04
- added J9: USART_LogicAnalyzer, symbol Connector_Generic:Conn_01x03
- MK1, MK2, MK3, MK4, MK5: symbol BPSDisplay-rescue:Mounting_Hole-Mechanical -> BPSDisplay-rescue:Mounting_Hole-Mechanical-BPSDisplay-rescue
Connections:
- wire segments 160 -> 165
Changed lines of the file:
@@
 ID_SD and ID_SC PINS:\nThese pins are reserved for HAT ID EEPROM.\n\nAt boot time this I2C interface will be\ninterrogated to look for an EEPROM\nthat identifes the attached board and\nallows automagic setup of the GPIOs\n(and optionally, Linux drivers).\n\nDO NOT USE these pins for anything other\nthan attaching an I2C ID EEPROM. Leave\nunconnected if ID EEPROM not required.
 $Comp
-L BPSDisplay-rescue:Mounting_Hole-Mechanical MK1
+L BPSDisplay-rescue:Mounting_Hole-Mechanical-BPSDisplay-rescue MK1
 U 1 1 5834FB2E
 P 3000 7200
@@
 $EndComp
 $Comp
-L BPSDisplay-rescue:Mounting_Hole-Mechanical MK2
+L BPSDisplay-rescue:Mounting_Hole-Mechanical-BPSDisplay-rescue MK2
 U 1 1 5834FBEF
 P 3450 7200
@@
 $EndComp
 $Comp
-L BPSDisplay-rescue:Mounting_Hole-Mechanical MK4
+L BPSDisplay-rescue:Mounting_Hole-Mechanical-BPSDisplay-rescue MK4
 U 1 1 5834FC19
 P 3000 7400
@@
 Text Label 7250 4500 2    50   ~ 0
 CAN2_RX
-Wire Wire Line
-	1900 3950 2400 3950
-Wire Wire Line
-	2400 4050 1900 4050
-Text Label 2400 3950 2    50   ~ 0
-CAN2_TX
-Text Label 2400 4050 2    50   ~ 0
-CAN2_RX
 $Comp
 L power:GND #PWR019
@@
 $EndComp
 Wire Wire Line
-	2000 4250 2000 4150
-Wire Wire Line
 	2000 4150 1900 4150
 Wire Wire Line
 	2250 3850 1900 3850
-$Comp
-L Connector_Generic:Conn_02x06_Counter_Clockwise J2
-U 1 1 5D725DDF
-P 9600 3350
-F 0 "J2" H 9650 3767 50  0000 C CNN
-F 1 "Conn_02x06_Counter_Clockwise" H 9650 3676 50  0000 C CNN
-F 2 "Connector_PinHeader_2.54mm:PinHeader_2x06_P2.54mm_Vertical" H 9600 3350 50  0001 C CNN
-F 3 "~" H 9600 3350 50  0001 C CNN
-	1    9600 3350
-	1    0    0    -1
-$EndComp
-$Comp
-L power:GND #PWR015
-U 1 1 5D7263C8
-P 8450 3150
-F 0 "#PWR015" H 8450 2900 50  0001 C CNN
-F 1 "GND" H 8455 2977 50  0000 C CNN
-F 2 "" H 8450 3150 50  0001 C CNN
-F 3 "" H 8450 3150 50  0001 C CNN
-	1    8450 3150
-	0    1    1    0
-$EndComp
-Wire Wire Line
-	8450 3150 9400 3150
 Text Notes 7550 2600 0    50   ~ 0
 DC
@@
 Text Notes 7550 2200 0    50   ~ 0
 SCK
-Wire Wire Line
-	9400 3250 8650 3250
-Wire Wire Line
-	9400 3350 8650 3350
-Wire Wire Line
-	8650 3450 9400 3450
-Wire Wire Line
-	9400 3550 8650 3550
-Wire Wire Line
-	8650 3650 9400 3650
-Wire Wire Line
-	9900 3250 10650 3250
-Wire Wire Line
-	10650 3150 9900 3150
-Text Label 8650 3450 0    50   ~ 0
-GPIO10(SPI0_MOSI)
-Text Label 8650 3350 0    50   ~ 0
-GPIO9(SPI0_MISO)
-Text Label 8650 3250 0    50   ~ 0
-GPIO11(SPI0_SCK)
-Text Label 8650 3550 0    50   ~ 0
-GPIO8(SPI0_CE_N)
-Text Label 8650 3650 0    50   ~ 0
-GPIO25(GEN6)
-Text Label 10650 3250 2    50   ~ 0
-GPIO17(GEN0)
-Text Label 10650 3150 2    50   ~ 0
-GPIO24(GEN5)
-Text Notes 8600 3650 2    50   ~ 0
+Text Notes 8700 5200 2    50   ~ 0
 DC
-Text Notes 10700 3250 0    50   ~ 0
+Text Notes 8550 5400 0    50   ~ 0
 RST
-Text Notes 10700 3150 0    50   ~ 0
+Text Notes 8550 5300 0    50   ~ 0
 BUSY
-Text Notes 8600 3550 2    50   ~ 0
+Text Notes 8450 4650 2    50   ~ 0
 CS
-Text Notes 8600 3450 2    50   ~ 0
+Text Notes 8500 4550 2    50   ~ 0
 MOSI
-Text Notes 8600 3350 2    50   ~ 0
+Text Notes 8500 4450 2    50   ~ 0
 MISO
-Text Notes 8600 3250 2    50   ~ 0
+Text Notes 8500 4350 2    50   ~ 0
 SCK
-Wire Wire Line
-	9900 3550 10400 3550
-Wire Wire Line
-	10400 3650 9900 3650
-Text Label 10400 3550 2    50   ~ 0
-CAN2_TX
-Text Label 10400 3650 2    50   ~ 0
-CAN2_RX
 Wire Wire Line
 	5350 3900 4850 3900
@@
 USART6_TX
 Text Label 4850 4000 0    50   ~ 0
-USART6_RX
-Wire Wire Line
-	9900 3350 10400 3350
-Wire Wire Line
-	10400 3450 9900 3450
-Text Label 10400 3350 2    50   ~ 0
-USART6_TX
-Text Label 10400 3450 2    50   ~ 0
 USART6_RX
 $Comp
@@
 NoConn ~ 5350 3500
 $Comp
-L BPSDisplay-rescue:Mounting_Hole-Mechanical MK3
+L BPSDisplay-rescue:Mounting_Hole-Mechanical-BPSDisplay-rescue MK3
 U 1 1 5D979DD2
 P 4650 7200
@@
 $EndComp
 $Comp
-L BPSDisplay-rescue:Mounting_Hole-Mechanical MK5
+L BPSDisplay-rescue:Mounting_Hole-Mechanical-BPSDisplay-rescue MK5
 U 1 1 5D97A2E5
 P 4650 7400
@@
 Wire Wire Line
 	2750 1100 2750 1200
+$Comp
+L power:PWR_FLAG #FLG0101
+U 1 1 5F790F74
+P 5150 2100
+F 0 "#FLG0101" H 5150 2175 50  0001 C CNN
+F 1 "PWR_FLAG" V 5150 2227 50  0000 L CNN
+F 2 "" H 5150 2100 50  0001 C CNN
+F 3 "~" H 5150 2100 50  0001 C CNN
+	1    5150 2100
+	0    -1   -1   0
+$EndComp
+Connection ~ 5150 2100
+$Comp
+L Connector_Generic:Conn_01x05 J7
+U 1 1 5F8B1965
+P 9650 4450
+F 0 "J7" H 9730 4492 50  0000 L CNN
+F 1 "SPI0_LogicAnalyzer" H 9730 4401 50  0000 L CNN
+F 2 "" H 9650 4450 50  0001 C CNN
+F 3 "~" H 9650 4450 50  0001 C CNN
+	1    9650 4450
+	1    0    0    -1
+$EndComp
+Text Label 8500 4350 0    50   ~ 0
+GPIO11(SPI0_SCK)
+Text Label 8500 4450 0    50   ~ 0
+GPIO9(SPI0_MISO)
+Text Label 8500 4550 0    50   ~ 0
+GPIO10(SPI0_MOSI)
+Text Label 8500 4650 0    50   ~ 0
+GPIO8(SPI0_CE_N)
+$Comp
+L BPSDisplay:GND #PWR020
+U 1 1 5F8C3D7F
+P 9400 4150
+F 0 "#PWR020" H 9400 3900 50  0001 C CNN
+F 1 "GND" H 9405 3977 50  0000 C CNN
+F 2 "" H 9400 4150 50  0000 C CNN
+F 3 "" H 9400 4150 50  0000 C CNN
+	1    9400 4150
+	-1   0    0    1
+$EndComp
+Wire Wire Line
+	9450 4250 9400 4250
+Wire Wire Line
+	9400 4250 9400 4150
+Wire Wire Line
+	9450 4450 8500 4450
+Wire Wire Line
+	9450 4350 8500 4350
+Wire Wire Line
+	9450 4550 8500 4550
+Wire Wire Line
+	9450 4650 8500 4650
+$Comp
+L Connector_Generic:Conn_01x04 J8
+U 1 1 5F9133E1
+P 9650 5200
+F 0 "J8" H 9730 5192 50  0000 L CNN
+F 1 "GEN_LogicAnalyzer" H 9730 5101 50  0000 L CNN
+F 2 "" H 9650 5200 50  0001 C CNN
+F 3 "~" H 9650 5200 50  0001 C CNN
+	1    9650 5200
+	1    0    0    -1
+$EndComp
+$Comp
+L BPSDisplay:GND #PWR022
+U 1 1 5F91429A
+P 9450 5000
+F 0 "#PWR022" H 9450 4750 50  0001 C CNN
+F 1 "GND" H 9455 4827 50  0000 C CNN
+F 2 "" H 9450 5000 50  0000 C CNN
+F 3 "" H 9450 5000 50  0000 C CNN
+	1    9450 5000
+	-1   0    0    1
+$EndComp
+Wire Wire Line
+	9450 5100 9450 5000
+Text Label 8750 5200 0    50   ~ 0
+GPIO25(GEN6)
+Text Label 8750 5300 0    50   ~ 0
+GPIO24(GEN5)
+Text Label 8750 5400 0    50   ~ 0
+GPIO17(GEN0)
+Wire Wire Line
+	9450 5200 8750 5200
+Wire Wire Line
+	9450 5300 8750 5300
+Wire Wire Line
+	9450 5400 8750 5400
+$Comp
+L Connector_Generic:Conn_01x03 J9
+U 1 1 5F937701
+P 9650 5950
+F 0 "J9" H 9730 5992 50  0000 L CNN
+F 1 "USART_LogicAnalyzer" H 9730 5901 50  0000 L CNN
+F 2 "" H 9650 5950 50  0001 C CNN
+F 3 "~" H 9650 5950 50  0001 C CNN
+	1    9650 5950
+	1    0    0    -1
+$EndComp
+$Comp
+L BPSDisplay:GND #PWR029
+U 1 1 5F937BE0
+P 9450 5750
+F 0 "#PWR029" H 9450 5500 50  0001 C CNN
+F 1 "GND" H 9455 5577 50  0000 C CNN
+F 2 "" H 9450 5750 50  0000 C CNN
+F 3 "" H 9450 5750 50  0000 C CNN
+	1    9450 5750
+	-1   0    0    1
+$EndComp
+Text Label 8750 5950 0    50   ~ 0
+USART6_TX
+Text Label 8750 6050 0    50   ~ 0
+USART6_RX
+Wire Wire Line
+	9450 5850 9450 5750
+Wire Wire Line
+	9450 5950 8750 5950
+Wire Wire Line
+	9450 6050 8750 6050
+Wire Wire Line
+	2000 4200 2000 4250
+Wire Wire Line
+	2000 4150 2000 4200
+Connection ~ 2000 4200
+Wire Wire Line
+	2550 4200 2000 4200
+Wire Wire Line
+	2550 3850 2550 4200
+Wire Wire Line
+	2700 3850 2550 3850
+Wire Wire Line
+	2700 4050 1900 4050
+Wire Wire Line
+	2700 3950 1900 3950
+$Comp
+L Connector_Generic:Conn_01x03 J6
+U 1 1 5F84797F
+P 2900 3950
+F 0 "J6" H 2980 3992 50  0000 L CNN
+F 1 "CAN_LogicAnalyzer" H 2980 3901 50  0000 L CNN
+F 2 "" H 2900 3950 50  0001 C CNN
+F 3 "~" H 2900 3950 50  0001 C CNN
+	1    2900 3950
+	1    0    0    -1
+$EndComp
+Text Label 2400 4050 2    50   ~ 0
+CAN2_RX
+Text Label 2400 3950 2    50   ~ 0
+CAN2_TX
 $EndSCHEMATC

Commit message: Added footprints to connectors
Made all connector footprints horizontal too
Parts:
- J6, J9: footprint (none) -> Connector_PinHeader_2.54mm:PinHeader_1x03_P2.54mm_Horizontal
- J7: footprint (none) -> Connector_PinHeader_2.54mm:PinHeader_1x05_P2.54mm_Horizontal
- J8: footprint (none) -> Connector_PinHeader_2.54mm:PinHeader_1x04_P2.54mm_Horizontal
- P1: footprint Connector_PinSocket_2.54mm:PinSocket_2x20_P2.54mm_Vertical -> Connector_PinSocket_2.54mm:PinSocket_2x20_P2.54mm_Horizontal
Changed lines of the file:
@@
 F 0 "P1" H 2300 3117 50  0000 C CNN
 F 1 "Conn_02x20_Odd_Even" H 2300 3026 50  0000 C CNN
-F 2 "Connector_PinSocket_2.54mm:PinSocket_2x20_P2.54mm_Vertical" H -2600 1050 50  0001 C CNN
+F 2 "Connector_PinSocket_2.54mm:PinSocket_2x20_P2.54mm_Horizontal" H -2600 1050 50  0001 C CNN
 F 3 "" H -2600 1050 50  0001 C CNN
 	1    2250 2000
@@
 F 0 "J7" H 9730 4492 50  0000 L CNN
 F 1 "SPI0_LogicAnalyzer" H 9730 4401 50  0000 L CNN
-F 2 "" H 9650 4450 50  0001 C CNN
+F 2 "Connector_PinHeader_2.54mm:PinHeader_1x05_P2.54mm_Horizontal" H 9650 4450 50  0001 C CNN
 F 3 "~" H 9650 4450 50  0001 C CNN
 	1    9650 4450
@@
 F 0 "J8" H 9730 5192 50  0000 L CNN
 F 1 "GEN_LogicAnalyzer" H 9730 5101 50  0000 L CNN
-F 2 "" H 9650 5200 50  0001 C CNN
+F 2 "Connector_PinHeader_2.54mm:PinHeader_1x04_P2.54mm_Horizontal" H 9650 5200 50  0001 C CNN
 F 3 "~" H 9650 5200 50  0001 C CNN
 	1    9650 5200
@@
 F 0 "J9" H 9730 5992 50  0000 L CNN
 F 1 "USART_LogicAnalyzer" H 9730 5901 50  0000 L CNN
-F 2 "" H 9650 5950 50  0001 C CNN
+F 2 "Connector_PinHeader_2.54mm:PinHeader_1x03_P2.54mm_Horizontal" H 9650 5950 50  0001 C CNN
 F 3 "~" H 9650 5950 50  0001 C CNN
 	1    9650 5950
@@
 F 0 "J6" H 2980 3992 50  0000 L CNN
 F 1 "CAN_LogicAnalyzer" H 2980 3901 50  0000 L CNN
-F 2 "" H 2900 3950 50  0001 C CNN
+F 2 "Connector_PinHeader_2.54mm:PinHeader_1x03_P2.54mm_Horizontal" H 2900 3950 50  0001 C CNN
 F 3 "~" H 2900 3950 50  0001 C CNN
 	1    2900 3950

Commit message: Updated footprints, re-routed traces
Changed logical analyzer footprints to vertical, changed 2x20 connector footprint back to the original footprint, changed CAN headers to vertical footprints.
Grouped components better so logic analyzer pins are closer to their corresponding pins on the microcontroller. Re-did traces accordingly.
Parts:
- J6, J9: footprint Connector_PinHeader_2.54mm:PinHeader_1x03_P2.54mm_Horizontal -> Connector_PinHeader_2.54mm:PinHeader_1x03_P2.54mm_Vertical
- J7: footprint Connector_PinHeader_2.54mm:PinHeader_1x05_P2.54mm_Horizontal -> Connector_PinHeader_2.54mm:PinHeader_1x05_P2.54mm_Vertical
- J8: footprint Connector_PinHeader_2.54mm:PinHeader_1x04_P2.54mm_Horizontal -> Connector_PinHeader_2.54mm:PinHeader_1x04_P2.54mm_Vertical
- P1: footprint Connector_PinSocket_2.54mm:PinSocket_2x20_P2.54mm_Horizontal -> Connector_PinSocket_2.54mm:PinSocket_2x20_P2.54mm_Vertical
Changed lines of the file:
@@
 F 0 "P1" H 2300 3117 50  0000 C CNN
 F 1 "Conn_02x20_Odd_Even" H 2300 3026 50  0000 C CNN
-F 2 "Connector_PinSocket_2.54mm:PinSocket_2x20_P2.54mm_Horizontal" H -2600 1050 50  0001 C CNN
+F 2 "Connector_PinSocket_2.54mm:PinSocket_2x20_P2.54mm_Vertical" H -2600 1050 50  0001 C CNN
 F 3 "" H -2600 1050 50  0001 C CNN
 	1    2250 2000
@@
 F 0 "J7" H 9730 4492 50  0000 L CNN
 F 1 "SPI0_LogicAnalyzer" H 9730 4401 50  0000 L CNN
-F 2 "Connector_PinHeader_2.54mm:PinHeader_1x05_P2.54mm_Horizontal" H 9650 4450 50  0001 C CNN
+F 2 "Connector_PinHeader_2.54mm:PinHeader_1x05_P2.54mm_Vertical" H 9650 4450 50  0001 C CNN
 F 3 "~" H 9650 4450 50  0001 C CNN
 	1    9650 4450
@@
 F 0 "J8" H 9730 5192 50  0000 L CNN
 F 1 "GEN_LogicAnalyzer" H 9730 5101 50  0000 L CNN
-F 2 "Connector_PinHeader_2.54mm:PinHeader_1x04_P2.54mm_Horizontal" H 9650 5200 50  0001 C CNN
+F 2 "Connector_PinHeader_2.54mm:PinHeader_1x04_P2.54mm_Vertical" H 9650 5200 50  0001 C CNN
 F 3 "~" H 9650 5200 50  0001 C CNN
 	1    9650 5200
@@
 F 0 "J9" H 9730 5992 50  0000 L CNN
 F 1 "USART_LogicAnalyzer" H 9730 5901 50  0000 L CNN
-F 2 "Connector_PinHeader_2.54mm:PinHeader_1x03_P2.54mm_Horizontal" H 9650 5950 50  0001 C CNN
+F 2 "Connector_PinHeader_2.54mm:PinHeader_1x03_P2.54mm_Vertical" H 9650 5950 50  0001 C CNN
 F 3 "~" H 9650 5950 50  0001 C CNN
 	1    9650 5950
@@
 F 0 "J6" H 2980 3992 50  0000 L CNN
 F 1 "CAN_LogicAnalyzer" H 2980 3901 50  0000 L CNN
-F 2 "Connector_PinHeader_2.54mm:PinHeader_1x03_P2.54mm_Horizontal" H 2900 3950 50  0001 C CNN
+F 2 "Connector_PinHeader_2.54mm:PinHeader_1x03_P2.54mm_Vertical" H 2900 3950 50  0001 C CNN
 F 3 "~" H 2900 3950 50  0001 C CNN
 	1    2900 3950

Commit message: Fixed traces
Got rid of traces with right angles, made labels on CAN headers vertical, made traces neater, added logo and picture of Dr. Hallock on back
Parts:
- added LOGO1: Logo_Placeholder, UTSVT_Special:UTSVT_Logo_Symbol, symbol utsvt-misc:Logo_Placeholder
- added LOGO2: Logo_Placeholder, UTSVT_Special:Hallock_Image_Tiny, symbol utsvt-misc:Logo_Placeholder
Changed lines of the file:
@@
 Text Label 2400 3950 2    50   ~ 0
 CAN2_TX
+$Comp
+L utsvt-misc:Logo_Placeholder LOGO1
+U 1 1 5F8BDCC5
+P 5500 7150
+F 0 "LOGO1" H 5500 7300 50  0001 C CNN
+F 1 "Logo_Placeholder" H 5640 7150 50  0000 L CNN
+F 2 "UTSVT_Special:UTSVT_Logo_Symbol" H 5500 7225 50  0001 C CNN
+F 3 "" H 5500 7225 50  0001 C CNN
+	1    5500 7150
+	1    0    0    -1
+$EndComp
+$Comp
+L utsvt-misc:Logo_Placeholder LOGO2
+U 1 1 5F8C0DEB
+P 5500 6800
+F 0 "LOGO2" H 5500 6950 50  0001 C CNN
+F 1 "Logo_Placeholder" H 5640 6800 50  0000 L CNN
+F 2 "UTSVT_Special:Hallock_Image_Tiny" H 5500 6875 50  0001 C CNN
+F 3 "" H 5500 6875 50  0001 C CNN
+	1    5500 6800
+	1    0    0    -1
+$EndComp
 $EndSCHEMATC
